Commit message: 

File: src/smartcar_description/urdf/smartcar_body.urdf.xacro (robot description, xacro)
@@ -26,5 +26,5 @@
                     <box size="0.25 0.16 0.05" />
                 </geometry>
-            </collicion>
+            </collision>
         </link>
         <link name="left_front_wheel">
@@ -60,10 +60,10 @@
             <inertial>
                 <origin xyz="0.08 -0.08 0.025" />
-                <mass value="1.0" />
+                <mass value="0.1" />
                 <inertia ixx="1.0" ixy="0.0" ixz="0.0" iyy="1.0" iyz="0.0" izz="1.0" />
             </inertial>
             <visual>
                 <geometry>
-                    <cylinder length="0.02" radius="0.05" />
+                    <cylinder length="0.02" radius="0.025" />
                 </geometry>
                 <material name="black">
@@ -89,10 +89,10 @@
             <inertial>
                 <origin xyz="-0.08 0.08 0.025" />
-                <mass value="1.0" />
+                <mass value="0.1" />
                 <inertia ixx="1.0" ixy="0.0" ixz="0.0" iyy="1.0" iyz="0.0" izz="0.0" />
             </inertial>
             <visual>
                 <geometry>
-                    <cylinder length="0.02" radius="0,05" />
+                    <cylinder length="0.02" radius="0.025" />
                 </geometry>
                 <material name="black">
@@ -111,5 +111,5 @@
             <parent link="base_link" />
             <child link="left_back_wheel" />
-            <origin rpy="0 1.57075 1.57.75" xyz="-0.08 0.08 0.25" />
+            <origin rpy="0 1.57075 1.57075" xyz="-0.08 0.08 0.25" />
             <limit effort="100" velocity="100" />
             <joint_properties damping="0.0" friction="0.0" />
@@ -117,11 +117,11 @@
         <link name="right_back_wheel">
             <inertial>
-                <origin rpy="0 1.57075 1.57075" xyz="-0.08 -0.08 0.025" />
-                <mass value="1.0" />
+                <origin xyz="-0.08 -0.08 0.025" />
+                <mass value="0.1" />
                 <inertia ixx="1.0" ixy="0.0" ixz="0.0" iyy="1.0" iyz="0.0" izz="1.0" />
             </inertial>
             <visual>
                 <geometry>
-                    <cylinder length="0.02" radius="0.05" />
+                    <cylinder length="0.02" radius="0.025" />
                 </geometry>
                 <material name="black">
@@ -132,5 +132,42 @@
                 <origin rpy="0 1.57075 1.57075" xyz="-0.08 -0.08 0.025" />
                 <geometry>
-                    <cylinder length="0.02" radius="0.05" />
+                    <cylinder length="0.02" radius="0.025" />
                 </geometry>
-            </collision>
+            </collision>
+        </link>
+        <joint name="right_back_wheel_joint" type="continuous">
+            <axis xyz="0 0 1" />
+            <parent link="base_link" />
+            <child link="right_back_wheel" />
+            <origin rpy="0 1.57075 1.57075" xyz="-0.08 -0.08 0.025" />
+            <limit effort="100" velocity="100" />
+            <joint_properties damping="0.0" friction="0.0" />
+        </joint>
+        <link name="head">
+            <inertial>
+                <origin xyz="0.08 0 0.08"/>
+                <mass value="0.1"/>
+                <inertia ixx="1.0" ixy="0.0" ixz="0.0" iyy="1.0" iyz="0.0" izz="1.0" />
+            </inertial>
+            <visual>
+                <geometry>
+                    <box size="0.02 0.03 0.03" />
+                </geometry>
+                <material name="white">
+                    <color rgba="1 1 1 1" />
+                </material>
+            </visual>
+            <collision>
+                <origin rpy="0 0 0 " xyz="0.08 0 0.08" />
+                <geometry>
+                    <box size="0.02 0.03 0.03" />
+                </geometry>
+            </collision>
+        </link>
+        <joint name="tobox" type="fixed">
+            <parent link="base_link" />
+            <child link="head" />
+            <origin rpy="0 0 0" xyz="0.08 0.08 0.08" />
+        </joint>
+    </xacro:macro>
+</robot>
