Commit message: smartcar simple functions

File: src/smartcar_description/urdf/gazebo.urdf.xacro (robot description, xacro)
@@ -1,5 +1,5 @@
-<?<?xml version="1.0"?>
+<?xml version="1.0"?>
 <robot xmlns:controller="http://playerstage.sourceforge.net/gazebo/xmlschema/#controller"
-    xmlns:interface="http://playerstage.sourceforge.net/gazebo/xmlchema/#interface"
+    xmlns:interface="http://playerstage.sourceforge.net/gazebo/xmlschema/#interface"
     xmlns:sensor="http://playerstage.sourceforge.net/gazebo/xmlschema/#sensor"
     xmlns:xacro="http://ros.org/wiki/xacro"

File: src/smartcar_description/urdf/smartcar.urdf.xacro (robot description, xacro)
@@ -1,3 +1,3 @@
-<?<?xml version="1.0"?>
+<?xml version="1.0"?>
 <robot name="smartcar"
     xmlns:xi="http://www.w3.org/2001/XInclude"

File: src/smartcar_description/urdf/smartcar_body.urdf.xacro (robot description, xacro)
@@ -169,5 +169,5 @@
             <parent link="base_link" />
             <child link="head" />
-            <origin rpy="0 0 0" xyz="0.08 0.08 0.08" />
+            <origin rpy="0 0 0" xyz="0.08 0 0.08" />
         </joint>
     </xacro:macro>

Commit message: simple functions

File: src/smartcar_description/urdf/gazebo.urdf.xacro (robot description, xacro)
@@ -1,5 +1,5 @@
-<?<?xml version="1.0"?>
+<?xml version="1.0"?>
 <robot xmlns:controller="http://playerstage.sourceforge.net/gazebo/xmlschema/#controller"
-    xmlns:interface="http://playerstage.sourceforge.net/gazebo/xmlchema/#interface"
+    xmlns:interface="http://playerstage.sourceforge.net/gazebo/xmlschema/#interface"
     xmlns:sensor="http://playerstage.sourceforge.net/gazebo/xmlschema/#sensor"
     xmlns:xacro="http://ros.org/wiki/xacro"
@@ -27,3 +27,3 @@
         </gazebo>
     </xacro:macro>
-</robot>>
+</robot>

File: src/smartcar_description/urdf/smartcar.urdf.xacro (robot description, xacro)
@@ -1,3 +1,3 @@
-<?<?xml version="1.0"?>
+<?xml version="1.0"?>
 <robot name="smartcar"
     xmlns:xi="http://www.w3.org/2001/XInclude"
@@ -13,5 +13,5 @@
     xmlns:renderable="http://playerstage.sourceforge.net/gazebo/xmlschema/#renderable"
     xmlns:physics="http://playerstage.sourceforge.net/gazebo/xmlschema/#physics"
-    xmlns:xacro="http://ros.org/wiki/xacro">
+    xmlns:xacro="http://ros.org/wiki/xacro" >
     <xacro:include filename="$(find smartcar_description)/urdf/smartcar_body.urdf.xacro" />
     <!--Body of SmartCar, with plates standoffs and Create (including sim sensor)-->

File: src/smartcar_description/urdf/smartcar_body.urdf.xacro (robot description, xacro)
@@ -17,5 +17,5 @@
                     <box size="0.25 0.16 0.05" />
                 </geometry>
-                <origin rpy="0 0 0" xyz="0 0 0.055" />
+                <origin xyz="0 0 0.055" />
                 <material name="blue">
                     <color rgba="0 0 0.8 1" />
@@ -23,5 +23,5 @@
             </visual>
             <collision>
-                <origin rpy="0 0 0" xyz="0 0 0.055" />
+                <origin xyz="0 0 0.055" />
                 <geometry>
                     <box size="0.25 0.16 0.05" />
@@ -33,5 +33,5 @@
                 <origin xyz="0.08 0.08 0.025" />
                 <mass value="0.1" />
-                <inertia ixx="1.0" ixy="0.0" ixz="0.0" iyy="1.0" iyz="0.0" izz="0.0" />
+                <inertia ixx="1.0" ixy="0.0" ixz="0.0" iyy="1.0" iyz="0.0" izz="1.0" />
             </inertial>
             <visual>
@@ -40,9 +40,8 @@
                 </geometry>
                 <material name="black">
-                    <color rgba=="0 0 0 1" />
+                    <color rgba="0 0 0 1" />
                 </material>
             </visual>
             <collision>
-                <origin rpy="0 1.57075 1.57075" xyz="0.08 0.08 0.025" />
                 <geometry>
                     <cylinder length="0.02" radius="0.025" />
@@ -73,5 +72,4 @@
             </visual>
             <collision>
-                <origin rpy="0 1.57075 1.57075" xyz="0.08 -0.08 0.025" />
                 <geometry>
                     <cylinder length="0.02" radius="0.025" />
@@ -112,5 +110,5 @@
             <parent link="base_link" />
             <child link="left_back_wheel" />
-            <origin rpy="0 1.57075 1.57075" xyz="-0.08 0.08 0.25" />
+            <origin rpy="0 1.57075 1.57075" xyz="-0.08 0.08 0.025" />
             <limit effort="100" velocity="100" />
             <joint_properties damping="0.0" friction="0.0" />
@@ -131,5 +129,4 @@
             </visual>
             <collision>
-                <origin rpy="0 1.57075 1.57075" xyz="-0.08 -0.08 0.025" />
                 <geometry>
                     <cylinder length="0.02" radius="0.025" />
@@ -160,5 +157,4 @@
             </visual>
             <collision>
-                <origin rpy="0 0 0 " xyz="0.08 0 0.08" />
                 <geometry>
                     <box size="0.02 0.03 0.03" />
@@ -169,5 +165,5 @@
             <parent link="base_link" />
             <child link="head" />
-            <origin rpy="0 0 0" xyz="0.08 0.08 0.08" />
+            <origin rpy="0 0 0" xyz="0.08 0 0.08" />
         </joint>
     </xacro:macro>
